Commit message: fix: URDF xacro 차체, LiDAR offset 값 수정

File: src/wave_rover_slam/urdf/wave_rover.urdf.xacro (robot description, xacro)
@@ -2,7 +2,7 @@
 <robot name="wave_rover" xmlns:xacro="http://www.ros.org/wiki/xacro">
   <!-- 차체 크기 상수 정의 (단위: m) -->
-  <xacro:property name="base_length" value="0.194"/>
+  <xacro:property name="base_length" value="0.250"/>
   <xacro:property name="base_width"  value="0.168"/>
-  <xacro:property name="base_height" value="0.100"/>
+  <xacro:property name="base_height" value="0.139"/>
   <!-- 타이어 크기 상수 정의 -->
   <xacro:property name="wheel_radius" value="0.040"/>
@@ -45,5 +45,5 @@
     <parent link="base_link"/>
     <child  link="laser"/>
-    <origin xyz="0.08 0 0.13" rpy="0 0 0"/>
+    <origin xyz="0.062 0 0.135" rpy="0 0 0"/>
   </joint>
   <link name="laser">

Commit message: fix: 차체 하드웨어 변경으로 인한 urdf 수정

File: src/wave_rover_slam/urdf/wave_rover.urdf.xacro (robot description, xacro)
@@ -2,7 +2,7 @@
 <robot name="wave_rover" xmlns:xacro="http://www.ros.org/wiki/xacro">
   <!-- 차체 크기 상수 정의 (단위: m) -->
-  <xacro:property name="base_length" value="0.250"/>
-  <xacro:property name="base_width"  value="0.168"/>
-  <xacro:property name="base_height" value="0.139"/>
+  <xacro:property name="base_length" value="0.183"/>
+  <xacro:property name="base_width"  value="0.170"/>
+  <xacro:property name="base_height" value="0.0885"/>
   <!-- 타이어 크기 상수 정의 -->
   <xacro:property name="wheel_radius" value="0.040"/>
@@ -45,5 +45,5 @@
     <parent link="base_link"/>
     <child  link="laser"/>
-    <origin xyz="0.062 0 0.135" rpy="0 0 0"/>
+    <origin xyz="0.09 0 0.12075" rpy="0 0 0"/>
   </joint>
   <link name="laser">
